Commit message: finished the urdf

File: install/kortex-gen3_description/share/kortex-gen3_description/urdf/arm.urdf (robot description, URDF)
Before this commit: robot kortex-gen3-lite, 6 links, 5 joints
Joints:
- joint arm_to_forearm: origin xyz=0 0.55 0 rpy=0 3.14 1.55 -> xyz=0 0.55 0 rpy=0 3.14 2.14
- joint forearm_to_upper_wrist: axis 0 1 0 -> 0 0 1; origin xyz=0 -0.46 -0.02 rpy=0 0 -1.57 -> xyz=0 -0.48 0 rpy=0 0 4.71
- joint shoulder_to_arm: origin xyz=0 0 0.20 rpy=1.57 0.38 0 -> xyz=0 0 0.20 rpy=1.57 0.78 0
- joint upper_wrist_to_lower_wrist: axis 1 0 0 -> 0 0 1; origin xyz=0.22 0 0 rpy=-3.14 4.71 3.14 -> xyz=0.22 0 0 rpy=3.14 1.57 0
